File: ORB/orb/orb.kicad_sch (KiCad schematic)
At the start: 11 parts, among them J1 Conn_01x02_Socket, J2 Conn_01x02_Socket, J3 Conn_01x02_Socket, J4 Conn_01x02_Socket, U1 Arduino_Nano, U3 4071

Commit message: Updated for 0.4.alpha release
Parts:
- removed E12, E20, E35, E6: MM1702A, Package_DIP:DIP-24_W10.16mm_Socket, symbol Sphere:MM1702A
- added D4: IN914, Diode_THT:D_DO-41_SOD81_P10.16mm_Horizontal, symbol Sphere:1N4001
- added D5, D6, D7: IN4001, Diode_THT:D_DO-41_SOD81_P10.16mm_Horizontal, symbol Sphere:1N4001
- added E12-1, E12-2, E12-3, E12-4, E20-1, E20-2, E20-3, E20-4, E35-1, E35-2, E35-3, E35-4, E6-2, E6-4: Conn_01x12_Pin, Connector_PinHeader_2.54mm:PinHeader_1x12_P2.54mm_Vertical, symbol Connector:Conn_01x12_Pin
- added E6-1, E6-3: E6-1C, Connector_PinHeader_2.54mm:PinHeader_1x12_P2.54mm_Vertical, symbol Connector:Conn_01x12_Pin
- D8: renamed from D1; value 1N4001 -> IN4001
- J1, J2, J3, J4: footprint Connector_PinHeader_1.00mm:PinHeader_1x02_P1.00mm_Vertical -> Connector_PinSocket_2.54mm:PinSocket_1x02_P2.54mm_Vertical
- U2: renamed from U3; footprint Connector_PinSocket_1.27mm:PinSocket_2x07_P1.27mm_Vertical -> Package_DIP:DIP-14_W7.62mm_Socket_LongPads
Connections:
- net at U1.10 (D7): now also E12-2.7 (Pin_7), E12-4.7 (Pin_7), E20-2.7 (Pin_7), E20-4.7 (Pin_7), E35-2.7 (Pin_7), E35-4.7 (Pin_7), E6-2.7 (Pin_7), E6-4.7 (Pin_7)
- net at U1.21 (A2/D16): now also E12-1.7 (Pin_7), E12-3.7 (Pin_7), E20-1.7 (Pin_7), E20-3.7 (Pin_7), E35-1.7 (Pin_7), E35-3.7 (Pin_7), E6-1.7 (Pin_7), E6-3.7 (Pin_7)
- net at U1.22 (A3/D17): now also E12-1.8 (Pin_8), E12-3.8 (Pin_8), E20-1.8 (Pin_8), E20-3.8 (Pin_8), E35-1.8 (Pin_8), E35-3.8 (Pin_8), E6-1.8 (Pin_8), E6-3.8 (Pin_8)
- net at U1.5 (D2): now also E12-2.2 (Pin_2), E12-4.2 (Pin_2), E20-2.2 (Pin_2), E20-4.2 (Pin_2), E35-2.2 (Pin_2), E35-4.2 (Pin_2), E6-2.2 (Pin_2), E6-4.2 (Pin_2)
- net at U1.6 (~D3): now also E12-2.3 (Pin_3), E12-4.3 (Pin_3), E20-2.3 (Pin_3), E20-4.3 (Pin_3), E35-2.3 (Pin_3), E35-4.3 (Pin_3), E6-2.3 (Pin_3), E6-4.3 (Pin_3)
- net at U1.7 (D4): now also E12-2.4 (Pin_4), E12-4.4 (Pin_4), E20-2.4 (Pin_4), E20-4.4 (Pin_4), E35-2.4 (Pin_4), E35-4.4 (Pin_4), E6-2.4 (Pin_4), E6-4.4 (Pin_4)
- net at U1.11 (D8): now also E12-2.8 (Pin_8), E12-4.8 (Pin_8), E20-2.8 (Pin_8), E20-4.8 (Pin_8), E35-2.8 (Pin_8), E35-4.8 (Pin_8), E6-2.8 (Pin_8), E6-4.8 (Pin_8)
- net at U1.8 (~D5): now also E12-2.5 (Pin_5), E12-4.5 (Pin_5), E20-2.5 (Pin_5), E20-4.5 (Pin_5), E35-2.5 (Pin_5), E35-4.5 (Pin_5), E6-2.5 (Pin_5), E6-4.5 (Pin_5)
- net at U1.9 (~D6): now also E12-2.6 (Pin_6), E12-4.6 (Pin_6), E20-2.6 (Pin_6), E20-4.6 (Pin_6), E35-2.6 (Pin_6), E35-4.6 (Pin_6), E6-2.6 (Pin_6), E6-4.6 (Pin_6)
- net at D8.2 (A), J4.2 (Pin_2): now also E12-1.1 (Pin_1), E12-3.1 (Pin_1), E20-1.1 (Pin_1), E20-3.1 (Pin_1), E35-1.1 (Pin_1), E35-3.1 (Pin_1), E6-1.1 (Pin_1), E6-3.1 (Pin_1)
- net at U1.12 (~D9): now also E12-2.9 (Pin_9), E12-4.9 (Pin_9), E20-2.9 (Pin_9), E20-4.9 (Pin_9), E35-2.9 (Pin_9), E35-4.9 (Pin_9), E6-2.9 (Pin_9), E6-4.9 (Pin_9)
- net at U1.13 (~D10): now also E12-2.10 (Pin_10), E12-4.10 (Pin_10), E20-2.10 (Pin_10), E20-4.10 (Pin_10), E35-2.10 (Pin_10), E35-4.10 (Pin_10), E6-2.10 (Pin_10), E6-4.10 (Pin_10)
- net at U1.14 (~D11): now also E12-2.11 (Pin_11), E12-4.11 (Pin_11), E20-2.11 (Pin_11), E20-4.11 (Pin_11), E35-2.11 (Pin_11), E35-4.11 (Pin_11), E6-2.11 (Pin_11), E6-4.11 (Pin_11)
- net at U1.15 (D12): now also E12-2.12 (Pin_12), E12-4.12 (Pin_12), E20-2.12 (Pin_12), E20-4.12 (Pin_12), E35-2.12 (Pin_12), E35-4.12 (Pin_12), E6-2.12 (Pin_12), E6-4.12 (Pin_12)
- net at U1.16 (D13): now also E12-1.4 (Pin_4), E12-3.4 (Pin_4), E20-1.4 (Pin_4), E20-3.4 (Pin_4), E35-1.4 (Pin_4), E35-3.4 (Pin_4), E6-1.4 (Pin_4), E6-3.4 (Pin_4)
- net at U1.19 (A0/D14): now also E12-1.5 (Pin_5), E12-3.5 (Pin_5), E20-1.5 (Pin_5), E20-3.5 (Pin_5), E35-1.5 (Pin_5), E35-3.5 (Pin_5), E6-1.5 (Pin_5), E6-3.5 (Pin_5)
- net at U1.20 (A1/D15): now also E12-1.6 (Pin_6), E12-3.6 (Pin_6), E20-1.6 (Pin_6), E20-3.6 (Pin_6), E35-1.6 (Pin_6), E35-3.6 (Pin_6), E6-1.6 (Pin_6), E6-3.6 (Pin_6)
- net at U2.1: now also E20-1.11 (Pin_11), E20-3.11 (Pin_11)
- net at U2.2: now also E12-1.11 (Pin_11), E12-3.11 (Pin_11)
- net at J1.2 (Pin_2), U1.29 (GND), U2.7 (VSS): now also D4.1 (K)
- net at J4.1 (Pin_1): now also D4.2 (A), D7.1 (K); no longer D8.1 (K)
- net at U2.6: now also E6-1.11 (Pin_11), E6-3.11 (Pin_11)
- new net: D6.1 (K), D7.2 (A)
- new net: D5.1 (K), D6.2 (A)
- new net: D5.2 (A), D8.1 (K)
Other:
- note added: "0.4 04-JUL-2024 A. Shapton Second production prototype in line with CPU/2 board"
- note added: "1"
- note added: "A1"
- note added: "A3"
- note added: "A4"
- note added: "A5"
- note added: "A6"
- note added: "A7"
- note added: "A8"
- note added: "Address Lines 0-8 addressPin[] {D9, D8, D7, D6, D5, D4, D3, D2} Data Lines 0-8 dataPin[] {D10, D11, D12, D13, A0, A1, A2, A3} Chip Select lines 0 & 1 chipSelectPin[] {A6, A7} Expansion EXP1_1 = 0; Pins for Expansion-1 EXP1_2 = 1; EXP2_1 = A4; Pins for Expansion-2 EXP2_2 = A5;"
- note added: "CS"
- note added: "D1"
- note added: "D2"
- note added: "D3"
- note added: "D4"
- note added: "D5"
- note added: "D6"
- note added: "D7"
- note added: "D8"
- note added: "E12 Connectors"
- note added: "E12 EPROM 2"
- note added: "E20 Connectors"
- note added: "E20 EPROM 3"
- note added: "E35 Connectors"
- note added: "E35 EPROM 4"
- note added: "E6 Connectors"
- note added: "E6 EPROM 1"
- note added: "MM1702A Socket spacing 9.8mm between sockets 15.24 mm between rows 2.54mm between pins"
- note added: "V_{DD}"
- note removed: "EPROM 1"
- note removed: "EPROM 2"
- note removed: "EPROM 3"
- note removed: "EPROM 4"
- note removed: "KEY"
- moved on the sheet: D8, U1, U2A, U2B, U2E
